File: fmcp_sma.sch (KiCad schematic (older format))
At the start: 62 parts, among them J101 Conn_Coaxial, J102 Conn_Coaxial, J103 FMCP_VITA57.4, J104 Conn_Coaxial, J105 Conn_Coaxial, J106 Conn_Coaxial, J107 Conn_Coaxial, J108 Conn_Coaxial, J109 Conn_Coaxial, J110 Conn_Coaxial, J111 Conn_Coaxial, J112 Conn_Coaxial, J113 Conn_Coaxial, J114 Conn_Coaxial, J115 Conn_Coaxial, J116 Conn_Coaxial, J117 Conn_Coaxial, J118 Conn_Coaxial, J119 Conn_Coaxial, J120 Conn_Coaxial, J121 Conn_Coaxial, J122 Conn_01x03_Male, U101 M24C02-FDW

Commit message: bom csv xml
Parts:
- J101, J102, J104, J105, J106, J107, J116, J117, J118, J119, J120, J121: rs# 253-0085 -> (none)
- J108, J109, J110, J111, J112, J113, J114, J115: manf (none) -> Amphenol RF; manf# (none) -> 132134RP
- R101, R102, R103, R104, R105, R106, R107, R108, R109, R110, R111, R112, R113: stock (none) -> AVT-IPE
- U101: manf (none) -> STMicroelectronics; manf# (none) -> M24C02-FDW6TP; rs# (none) -> 190-7599
Changed lines of the file:
@@
 F 3 "~" H 9750 14900 50  0001 C CNN
 F 4 "DNP" H 9820 14809 50  0000 L CNN "DNP"
+F 5 "AVT-IPE" H 9750 14900 50  0001 C CNN "stock"
 	1    9750 14900
 	1    0    0    -1
@@
 F 3 "~" H 10050 14900 50  0001 C CNN
 F 4 "DNP" H 10120 14809 50  0000 L CNN "DNP"
+F 5 "AVT-IPE" H 10050 14900 50  0001 C CNN "stock"
 	1    10050 14900
 	1    0    0    -1
@@
 F 2 "Connector_Coaxial:SMA_Amphenol_132134_Vertical" H 17200 2600 50  0001 C CNN
 F 3 " ~" H 17200 2600 50  0001 C CNN
-F 4 "" H 17200 2600 50  0001 C CNN "manf"
-F 5 "" H 17200 2600 50  0001 C CNN "manf#"
+F 4 "Amphenol RF" H 17200 2600 50  0001 C CNN "manf"
+F 5 "132134RP" H 17200 2600 50  0001 C CNN "manf#"
 F 6 "" H 17200 2600 50  0001 C CNN "mouser#"
 F 7 "" H 17200 2600 50  0001 C CNN "digikey#"
@@
 F 2 "Connector_Coaxial:SMA_Amphenol_132134_Vertical" H 16800 2700 50  0001 C CNN
 F 3 " ~" H 16800 2700 50  0001 C CNN
-F 4 "" H 16800 2700 50  0001 C CNN "manf"
-F 5 "" H 16800 2700 50  0001 C CNN "manf#"
+F 4 "Amphenol RF" H 16800 2700 50  0001 C CNN "manf"
+F 5 "132134RP" H 16800 2700 50  0001 C CNN "manf#"
 F 6 "" H 16800 2700 50  0001 C CNN "mouser#"
 F 7 "" H 16800 2700 50  0001 C CNN "digikey#"
@@
 F 6 "" H 11100 5400 50  0001 C CNN "mouser#"
 F 7 "" H 11100 5400 50  0001 C CNN "digikey#"
-F 8 "253-0085" H 11100 5400 50  0001 C CNN "rs#"
+F 8 "" H 11100 5400 50  0001 C CNN "rs#"
 	1    11100 5400
 	1    0    0    -1
@@
 F 6 "" H 10700 5500 50  0001 C CNN "mouser#"
 F 7 "" H 10700 5500 50  0001 C CNN "digikey#"
-F 8 "253-0085" H 10700 5500 50  0001 C CNN "rs#"
+F 8 "" H 10700 5500 50  0001 C CNN "rs#"
 	1    10700 5500
 	1    0    0    -1
@@
 F 2 "Connector_Coaxial:SMA_Amphenol_132134_Vertical" H 1250 8850 50  0001 C CNN
 F 3 " ~" H 1250 8850 50  0001 C CNN
-F 4 "" H 1250 8850 50  0001 C CNN "manf"
-F 5 "" H 1250 8850 50  0001 C CNN "manf#"
+F 4 "Amphenol RF" H 1250 8850 50  0001 C CNN "manf"
+F 5 "132134RP" H 1250 8850 50  0001 C CNN "manf#"
 F 6 "" H 1250 8850 50  0001 C CNN "mouser#"
 F 7 "" H 1250 8850 50  0001 C CNN "digikey#"
@@
 F 2 "Connector_Coaxial:SMA_Amphenol_132134_Vertical" H 1650 8950 50  0001 C CNN
 F 3 " ~" H 1650 8950 50  0001 C CNN
-F 4 "" H 1650 8950 50  0001 C CNN "manf"
-F 5 "" H 1650 8950 50  0001 C CNN "manf#"
+F 4 "Amphenol RF" H 1650 8950 50  0001 C CNN "manf"
+F 5 "132134RP" H 1650 8950 50  0001 C CNN "manf#"
 F 6 "" H 1650 8950 50  0001 C CNN "mouser#"
 F 7 "" H 1650 8950 50  0001 C CNN "digikey#"
@@
 F 6 "" H 11600 3500 50  0001 C CNN "mouser#"
 F 7 "" H 11600 3500 50  0001 C CNN "digikey#"
-F 8 "253-0085" H 11600 3500 50  0001 C CNN "rs#"
+F 8 "" H 11600 3500 50  0001 C CNN "rs#"
 	1    11600 3500
 	1    0    0    -1
@@
 F 6 "" H 12000 3400 50  0001 C CNN "mouser#"
 F 7 "" H 12000 3400 50  0001 C CNN "digikey#"
-F 8 "253-0085" H 12000 3400 50  0001 C CNN "rs#"
+F 8 "" H 12000 3400 50  0001 C CNN "rs#"
 	1    12000 3400
 	1    0    0    -1
@@
 F 2 "Package_SO:TSSOP-8_4.4x3mm_P0.65mm" H 8750 15600 50  0001 C CNN
 F 3 "http://www.st.com/content/ccc/resource/technical/document/datasheet/b0/d8/50/40/5a/85/49/6f/DM00071904.pdf/files/DM00071904.pdf/jcr:content/translations/en.DM00071904.pdf" H 8800 14750 50  0001 C CNN
+F 4 "    STMicroelectronics" H 8750 15250 50  0001 C CNN "manf"
+F 5 "M24C02-FDW6TP" H 8750 15250 50  0001 C CNN "manf#"
+F 6 "190-7599" H 8750 15250 50  0001 C CNN "rs#"
 	1    8750 15250
 	1    0    0    -1
@@
 F 2 "Connector_Coaxial:SMA_Amphenol_132134_Vertical" H 2100 9150 50  0001 C CNN
 F 3 " ~" H 2100 9150 50  0001 C CNN
-F 4 "" H 2100 9150 50  0001 C CNN "manf"
-F 5 "" H 2100 9150 50  0001 C CNN "manf#"
+F 4 "Amphenol RF" H 2100 9150 50  0001 C CNN "manf"
+F 5 "132134RP" H 2100 9150 50  0001 C CNN "manf#"
 F 6 "" H 2100 9150 50  0001 C CNN "mouser#"
 F 7 "" H 2100 9150 50  0001 C CNN "digikey#"
@@
 F 2 "Connector_Coaxial:SMA_Amphenol_132134_Vertical" H 2500 9250 50  0001 C CNN
 F 3 " ~" H 2500 9250 50  0001 C CNN
-F 4 "" H 2500 9250 50  0001 C CNN "manf"
-F 5 "" H 2500 9250 50  0001 C CNN "manf#"
+F 4 "Amphenol RF" H 2500 9250 50  0001 C CNN "manf"
+F 5 "132134RP" H 2500 9250 50  0001 C CNN "manf#"
 F 6 "" H 2500 9250 50  0001 C CNN "mouser#"
 F 7 "" H 2500 9250 50  0001 C CNN "digikey#"
@@
 F 2 "Connector_Coaxial:SMA_Amphenol_132134_Vertical" H 9500 8950 50  0001 C CNN
 F 3 " ~" H 9500 8950 50  0001 C CNN
-F 4 "" H 9500 8950 50  0001 C CNN "manf"
-F 5 "" H 9500 8950 50  0001 C CNN "manf#"
+F 4 "Amphenol RF" H 9500 8950 50  0001 C CNN "manf"
+F 5 "132134RP" H 9500 8950 50  0001 C CNN "manf#"
 F 6 "" H 9500 8950 50  0001 C CNN "mouser#"
 F 7 "" H 9500 8950 50  0001 C CNN "digikey#"
@@
 F 2 "Connector_Coaxial:SMA_Amphenol_132134_Vertical" H 9100 9050 50  0001 C CNN
 F 3 " ~" H 9100 9050 50  0001 C CNN
-F 4 "" H 9100 9050 50  0001 C CNN "manf"
-F 5 "" H 9100 9050 50  0001 C CNN "manf#"
+F 4 "Amphenol RF" H 9100 9050 50  0001 C CNN "manf"
+F 5 "132134RP" H 9100 9050 50  0001 C CNN "manf#"
 F 6 "" H 9100 9050 50  0001 C CNN "mouser#"
 F 7 "" H 9100 9050 50  0001 C CNN "digikey#"
@@
 F 6 "" H 22300 13350 50  0001 C CNN "mouser#"
 F 7 "" H 22300 13350 50  0001 C CNN "digikey#"
-F 8 "253-0085" H 22300 13350 50  0001 C CNN "rs#"
+F 8 "" H 22300 13350 50  0001 C CNN "rs#"
 	1    22300 13350
 	1    0    0    -1
@@
 F 6 "" H 19100 13350 50  0001 C CNN "mouser#"
 F 7 "" H 19100 13350 50  0001 C CNN "digikey#"
-F 8 "253-0085" H 19100 13350 50  0001 C CNN "rs#"
+F 8 "" H 19100 13350 50  0001 C CNN "rs#"
 	1    19100 13350
 	-1   0    0    -1
@@
 F 6 "" H 22300 14100 50  0001 C CNN "mouser#"
 F 7 "" H 22300 14100 50  0001 C CNN "digikey#"
-F 8 "253-0085" H 22300 14100 50  0001 C CNN "rs#"
+F 8 "" H 22300 14100 50  0001 C CNN "rs#"
 	1    22300 14100
 	1    0    0    -1
@@
 F 6 "" H 19100 14100 50  0001 C CNN "mouser#"
 F 7 "" H 19100 14100 50  0001 C CNN "digikey#"
-F 8 "253-0085" H 19100 14100 50  0001 C CNN "rs#"
+F 8 "" H 19100 14100 50  0001 C CNN "rs#"
 	1    19100 14100
 	-1   0    0    -1
@@
 F 2 "Resistor_SMD:R_0201_0603Metric" V 9330 3900 50  0001 C CNN
 F 3 "~" H 9400 3900 50  0001 C CNN
+F 4 "AVT-IPE" H 9400 3900 50  0001 C CNN "stock"
 	1    9400 3900
 	0    1    1    0
@@
 F 2 "Resistor_SMD:R_0201_0603Metric" V 9330 3800 50  0001 C CNN
 F 3 "~" H 9400 3800 50  0001 C CNN
+F 4 "AVT-IPE" H 9400 3800 50  0001 C CNN "stock"
 	1    9400 3800
 	0    1    1    0
@@
 F 6 "" H 11100 3800 50  0001 C CNN "mouser#"
 F 7 "" H 11100 3800 50  0001 C CNN "digikey#"
-F 8 "253-0085" H 11100 3800 50  0001 C CNN "rs#"
+F 8 "" H 11100 3800 50  0001 C CNN "rs#"
 	1    11100 3800
 	1    0    0    -1
@@
 F 6 "" H 10700 3900 50  0001 C CNN "mouser#"
 F 7 "" H 10700 3900 50  0001 C CNN "digikey#"
-F 8 "253-0085" H 10700 3900 50  0001 C CNN "rs#"
+F 8 "" H 10700 3900 50  0001 C CNN "rs#"
 	1    10700 3900
 	1    0    0    -1
@@
 F 2 "Resistor_SMD:R_0201_0603Metric" V 15730 2700 50  0001 C CNN
 F 3 "~" H 15800 2700 50  0001 C CNN
+F 4 "AVT-IPE" H 15800 2700 50  0001 C CNN "stock"
 	1    15800 2700
 	0    1    1    0
@@
 F 2 "Resistor_SMD:R_0201_0603Metric" V 15730 2600 50  0001 C CNN
 F 3 "~" H 15800 2600 50  0001 C CNN
+F 4 "AVT-IPE" H 15800 2600 50  0001 C CNN "stock"
 	1    15800 2600
 	0    1    1    0
@@
 F 2 "Resistor_SMD:R_0201_0603Metric" V 3730 9250 50  0001 C CNN
 F 3 "~" H 3800 9250 50  0001 C CNN
+F 4 "AVT-IPE" H 3800 9250 50  0001 C CNN "stock"
 	1    3800 9250
 	0    -1   1    0
@@
 F 2 "Resistor_SMD:R_0201_0603Metric" V 3730 9150 50  0001 C CNN
 F 3 "~" H 3800 9150 50  0001 C CNN
+F 4 "AVT-IPE" H 3800 9150 50  0001 C CNN "stock"
 	1    3800 9150
 	0    -1   1    0
@@
 F 2 "Resistor_SMD:R_0201_0603Metric" V 9330 5500 50  0001 C CNN
 F 3 "~" H 9400 5500 50  0001 C CNN
+F 4 "AVT-IPE" H 9400 5500 50  0001 C CNN "stock"
 	1    9400 5500
 	0    -1   1    0
@@
 F 2 "Resistor_SMD:R_0201_0603Metric" V 9330 5400 50  0001 C CNN
 F 3 "~" H 9400 5400 50  0001 C CNN
+F 4 "AVT-IPE" H 9400 5400 50  0001 C CNN "stock"
 	1    9400 5400
 	0    -1   1    0
@@
 F 2 "Resistor_SMD:R_0201_0603Metric" V 21430 14100 50  0001 C CNN
 F 3 "~" H 21500 14100 50  0001 C CNN
+F 4 "AVT-IPE" H 21500 14100 50  0001 C CNN "stock"
 	1    21500 14100
 	0    1    1    0
@@
 F 2 "Resistor_SMD:R_0201_0603Metric" V 21430 13350 50  0001 C CNN
 F 3 "~" H 21500 13350 50  0001 C CNN
+F 4 "AVT-IPE" H 21500 13350 50  0001 C CNN "stock"
 	1    21500 13350
 	0    1    1    0
@@
 F 2 "Resistor_SMD:R_0603_1608Metric" V 21230 1700 50  0001 C CNN
 F 3 "~" H 21300 1700 50  0001 C CNN
+F 4 "AVT-IPE" H 21300 1700 50  0001 C CNN "stock"
 	1    21300 1700
 	1    0    0    -1
@@
 F 6 "" H 22300 12000 50  0001 C CNN "mouser#"
 F 7 "" H 22300 12000 50  0001 C CNN "digikey#"
-F 8 "253-0085" H 22300 12000 50  0001 C CNN "rs#"
+F 8 "" H 22300 12000 50  0001 C CNN "rs#"
 	1    22300 12000
 	1    0    0    -1
@@
 F 6 "" H 19100 12000 50  0001 C CNN "mouser#"
 F 7 "" H 19100 12000 50  0001 C CNN "digikey#"
-F 8 "253-0085" H 19100 12000 50  0001 C CNN "rs#"
+F 8 "" H 19100 12000 50  0001 C CNN "rs#"
 	1    19100 12000
 	-1   0    0    -1
